File: control_unit/control_unit.kicad_sch (KiCad schematic)
At the start: 105 parts, among them J1 Conn_01x02_Pin, J4 Conn_01x04_Pin, J5 BLDC1, J7 BLDC2, J8 BLDC3, J9 BLDC4, Q3 2N7002, Q4 2N7002, U14 MCP2515-xSO, U15 BNO055 DIP, U3 ATA6561-GAQW-N, Y1 8M

Commit message: OKL[200~過渡応答を
Parts:
- renumbered Cbst to Cbst1, Css to Css1, Cvcc to Cvcc1, LED_BNO to LED_BNO1, R_CAN to R_CAN1, Rilim to Rilim1, Rpg to Rpg1, Rt to Rt1
Changed lines of the file:
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@@
 		(dnp no)
 		(fields_autoplaced yes)
-		(property "Reference" "R_CAN"
+		(property "Reference" "R_CAN1"
 			(at 398.78 60.9599 0)
 			(effects
@@
 			(project ""
 				(path "/37a62e38-d605-4440-86b8-fb3d0940d64a"
-					(reference "R_CAN")
+					(reference "R_CAN1")
 					(unit 1)
 				)
@@
 		(on_board yes)
 		(dnp no)
-		(property "Reference" "LED_BNO"
+		(property "Reference" "LED_BNO1"
 			(at 175.26 123.444 90)
 			(effects
@@
 			(project "control_unit"
 				(path "/37a62e38-d605-4440-86b8-fb3d0940d64a"
-					(reference "LED_BNO")
+					(reference "LED_BNO1")
 					(unit 1)
 				)
@@
 		(on_board yes)
 		(dnp no)
-		(property "Reference" "Rilim"
+		(property "Reference" "Rilim1"
 			(at 121.158 70.104 0)
 			(effects
@@
 			(project ""
 				(path "/37a62e38-d605-4440-86b8-fb3d0940d64a"
-					(reference "Rilim")
+					(reference "Rilim1")
 					(unit 1)
 				)
@@
 		(dnp no)
 		(fields_autoplaced yes)
-		(property "Reference" "Cvcc"
+		(property "Reference" "Cvcc1"
 			(at 114.3 81.2799 0)
 			(effects
@@
 			(project ""
 				(path "/37a62e38-d605-4440-86b8-fb3d0940d64a"
-					(reference "Cvcc")
+					(reference "Cvcc1")
 					(unit 1)
 				)
@@
 		(dnp no)
 		(fields_autoplaced yes)
-		(property "Reference" "Cbst"
+		(property "Reference" "Cbst1"
 			(at 114.3 50.8 90)
 			(effects
@@
 			(project ""
 				(path "/37a62e38-d605-4440-86b8-fb3d0940d64a"
-					(reference "Cbst")
+					(reference "Cbst1")
 					(unit 1)
 				)
@@
 		(on_board yes)
 		(dnp no)
-		(property "Reference" "Css"
+		(property "Reference" "Css1"
 			(at 76.708 53.086 90)
 			(effects
@@
 			(project "control_unit"
 				(path "/37a62e38-d605-4440-86b8-fb3d0940d64a"
-					(reference "Css")
+					(reference "Css1")
 					(unit 1)
 				)
@@
 		(on_board yes)
 		(dnp no)
-		(property "Reference" "Rpg"
+		(property "Reference" "Rpg1"
 			(at 86.36 85.09 90)
 			(effects
@@
 			(project ""
 				(path "/37a62e38-d605-4440-86b8-fb3d0940d64a"
-					(reference "Rpg")
+					(reference "Rpg1")
 					(unit 1)
 				)
@@
 		(on_board yes)
 		(dnp no)
-		(property "Reference" "Rt"
+		(property "Reference" "Rt1"
 			(at 72.136 49.53 90)
 			(effects
@@
 			(project ""
 				(path "/37a62e38-d605-4440-86b8-fb3d0940d64a"
-					(reference "Rt")
+					(reference "Rt1")
 					(unit 1)
 				)

Commit message: 制御基板配線開始
Parts:
- removed Cin13, Cin14, Cin15, Cin16, Cin17: 10u, Capacitor_SMD:C_1210_3225Metric_Pad1.33x2.70mm_HandSolder, symbol Device:C
- removed J9: BLDC4, Connector_PinHeader_2.54mm:PinHeader_1x03_P2.54mm_Vertical, symbol Connector:Conn_01x03_Pin
- removed JP1: SolderJumper_2_Bridged, symbol Jumper:SolderJumper_2_Bridged
- removed U10, U11, U12, U13, U6, U7, U8, U9: ~, basic_parts:SOT-23-5_L3.0-W1.7-P0.95-LS2.8-BR, symbol basic_parts:MCP1402T-E/OT
- removed U4: ~, basic_parts:wetness sensor, symbol basic_parts:wetness_sensor
- added Cout1: 100p, Capacitor_SMD:C_0603_1608Metric, symbol Device:C
- added Cout2: 0.1u, Capacitor_SMD:C_0603_1608Metric, symbol Device:C
- added Cout3: 47u, Capacitor_SMD:C_1210_3225Metric, symbol Device:C
- added J2: Conn_01x02_Socket, Connector_JST:JST_VH_B2P-VH_1x02_P3.96mm_Vertical, symbol Connector:Conn_01x02_Socket
- added J6: BLDC1, Connector_PinHeader_2.54mm:PinHeader_1x03_P2.54mm_Vertical, symbol Connector:Conn_01x03_Pin
- added JP1: Jumper_2_Bridged, TestPoint:TestPoint_2Pads_Pitch2.54mm_Drill0.8mm, symbol Jumper:Jumper_2_Bridged
- added M1: Motor_Servo, Connector_PinHeader_2.54mm:PinHeader_1x03_P2.54mm_Vertical, symbol Motor:Motor_Servo
- added TP1: TestPoint, Connector_Pin:Pin_D0.7mm_L6.5mm_W1.8mm_FlatFork, symbol Connector:TestPoint
- C2, C3: footprint (none) -> Capacitor_SMD:C_0603_1608Metric
- Cbst1, Css1: footprint (none) -> Capacitor_SMD:C_0603_1608Metric; LCSC (none) -> C14663
- Cc1: value 4.7n -> 5.6n; footprint (none) -> Capacitor_SMD:C_0603_1608Metric
- Cc2: value 0.15n -> 82p; footprint (none) -> Capacitor_SMD:C_0603_1608Metric
- Cc3: value 2.2n -> 1500p; footprint (none) -> Capacitor_SMD:C_0603_1608Metric
- Cin1, Cin10, Cin11, Cin12, Cin2, Cin3, Cin4, Cin5, Cin6, Cin7, Cin8, Cin9: footprint Capacitor_SMD:C_1210_3225Metric_Pad1.33x2.70mm_HandSolder -> Capacitor_SMD:C_1210_3225Metric
- Cvcc1: footprint (none) -> Capacitor_SMD:C_0603_1608Metric; LCSC (none) -> C23630
- Cvin1: renamed from C1; footprint (none) -> Capacitor_SMD:C_0603_1608Metric; LCSC (none) -> C14663
- J4: footprint Connector_PinHeader_2.54mm:PinHeader_1x04_P2.54mm_Vertical -> Connector_JST:JST_XH_B4B-XH-A_1x04_P2.50mm_Vertical
- J7: value BLDC2 -> BLDC1
- J8: value BLDC3 -> BLDC1
- L2: footprint (none) -> basic_parts:IND-SMD_L13.8-W12.6
- LED_BNO1, LED_ESC_1, LED_ESC_2, LED_ESC_3, LED_ESC_4, LED_ESC_5: footprint (none) -> LED_SMD:LED_1206_3216Metric
- R1: value 100k -> 20m; footprint (none) -> Diode_SMD:D_2010_5025Metric_Pad1.52x2.65mm_HandSolder
- R14, R15, R2, R3, R4, R5, R_CAN1, R_tx0, R_tx1, R_tx2, R_tx3: footprint (none) -> Resistor_SMD:R_0603_1608Metric
- Rc1: value 5.6k -> 10k; footprint (none) -> Resistor_SMD:R_0603_1608Metric_Pad0.98x0.95mm_HandSolder; LCSC (none) -> C25804
- Rc2: value 600 -> 560; footprint (none) -> Resistor_SMD:R_0603_1608Metric_Pad0.98x0.95mm_HandSolder; LCSC (none) -> C23204
- Rfb1: footprint (none) -> Resistor_SMD:R_0603_1608Metric_Pad0.98x0.95mm_HandSolder; LCSC (none) -> C25810
- Rfb2: footprint (none) -> Resistor_SMD:R_0603_1608Metric_Pad0.98x0.95mm_HandSolder; LCSC (none) -> C22978
- Rilim1: footprint (none) -> Resistor_SMD:R_0603_1608Metric; LCSC (none) -> C17471
- Rpg1: footprint (none) -> Resistor_SMD:R_0603_1608Metric; LCSC (none) -> C23196
- Rt1: footprint (none) -> Resistor_SMD:R_0603_1608Metric; LCSC (none) -> C4216
- Ruv1: footprint (none) -> Resistor_SMD:R_0603_1608Metric; LCSC (none) -> C23242
- Ruv2: footprint (none) -> Resistor_SMD:R_0603_1608Metric; LCSC (none) -> C22790
- U5: LCSC (none) -> C2876740
- Y1: footprint (none) -> Crystal:Crystal_SMD_HC49-SD
- renumbered Cout1 to Cout4, Cout2 to Cout5, Cout3 to Cout6, Cout4 to Cout7
Connections:
- net SERVO_LOGIC is gone; now on an unnamed net: D1.1 (K)
- net +24V: now also R1.2; no longer C2.1, C3.1, Cin1.2, Cin10.2, Cin11.2, Cin12.2, Cin2.2, Cin3.2, Cin4.2, Cin5.2, Cin6.2, Cin7.2, Cin8.2, Cin9.2, Cout4.2, Cout5.2, Cout6.2, Cout7.2, Css1.1, Cvcc1.2, Cvin1.2, D8.1 (K), J1.2 (Pin_2), J5.3 (Pin_3), J7.3 (Pin_3), J8.3 (Pin_3), LED_BNO1.1 (K), LED_ESC_1.1 (K), LED_ESC_2.1 (K), LED_ESC_3.1 (K), LED_ESC_4.1 (K), LED_ESC_5.1 (K), Q2.3 (S), Q3.2 (S), Q4.2 (S), R13.2, Rfb2.1, Rt1.1, Ruv2.2, U1.2 (GND), U14.9 (VSS), U15.2 (GND), U15.7 (GND), U2.14 (GND), U2.20 (GND), U2.25 (GND), U2.30 (GND), U2.34 (GND), U2.39 (GND), U2.6 (GND), U2.9 (GND), U3.2 (GND), U3.8 (STBY), U5.12 (PGND), U5.15 (EP), U5.16 (NC), U5.21 (EP), U5.6 (AGND), U5.8 (SYNCIN)
- net +3.3V: no longer R1.2
- net +5.1V: now also Cout1.2, Cout2.2, Cout3.1
- net +5V: now also M1.2 (+); no longer D1.2 (A)
- net BLDC1_RP4: now also J5.1 (Pin_1)
- net BLDC2_RP4: now also J6.1 (Pin_1)
- net BLDC3_RP4: now also J7.1 (Pin_1)
- net BLDC4_RP4: now also J8.1 (Pin_1)
- net PGOOD: now also TP1.1
- net at R2.1: now also J5.2 (Pin_2); no longer LED_ESC_1.2 (A)
- net at R2.2: now also LED_ESC_1.2 (A); no longer J5.2 (Pin_2)
- net at LED_ESC_2.2 (A): now also R3.2; no longer R3.1
- net at R_CAN1.2: now also JP1.2 (B)
- net at J8.2 (Pin_2): now also R5.1; no longer R4.2
- net SERVO2: now reaches U2.33 (GPIO13(PWM1))
- net SERVO2: now also J4.2 (Pin_2)
- net SERVO4: now reaches J4.4 (Pin_4)
- net SERVO4: now also U2.18 (GPIO24)
- net at LED_ESC_4.2 (A): now also R5.2; no longer R5.1
- net SERVO1: now reaches J4.1 (Pin_1)
- net SERVO1: now also U2.32 (GPIO12(PWM0))
- net SERVO3: now reaches J4.3 (Pin_3)
- net SERVO3: now also U2.16 (GPIO23)
- net at R4.1: now also J7.2 (Pin_2); no longer LED_ESC_3.2 (A)
- net at R1.1: no longer U2.37 (GPIO26)
- net at U3.6 (CANL): now also JP1.1 (A)
- net GND: now reaches U5.9 (NC)
- net GND: now also C2.1, C3.1, Cin1.2, Cin10.2, Cin11.2, Cin12.2, Cin2.2, Cin3.2, Cin4.2, Cin5.2, Cin6.2, Cin7.2, Cin8.2, Cin9.2, Cout4.2, Cout5.2, Cout6.2, Cout7.2, Css1.1, Cvcc1.2, Cvin1.2, D8.1 (K), J1.2 (Pin_2), J5.3 (Pin_3), J7.3 (Pin_3), J8.3 (Pin_3), LED_BNO1.1 (K), LED_ESC_1.1 (K), LED_ESC_2.1 (K), LED_ESC_3.1 (K), LED_ESC_4.1 (K), LED_ESC_5.1 (K), Q2.3 (S), Q3.2 (S), Q4.2 (S), R13.2, Rfb2.1, Rt1.1, Ruv2.2, U1.2 (GND), U14.9 (VSS), U15.2 (GND), U15.7 (GND), U2.14 (GND), U2.20 (GND), U2.25 (GND), U2.30 (GND), U2.34 (GND), U2.39 (GND), U2.6 (GND), U2.9 (GND), U3.2 (GND), U3.8 (STBY), U5.12 (PGND), U5.15 (EP), U5.16 (NC), U5.21 (EP), U5.6 (AGND), U5.8 (SYNCIN), Cout1.1, Cout2.1, Cout3.2, J2.2 (Pin_2), J6.3 (Pin_3), M1.3 (-)
- new net: J6.2 (Pin_2), R3.1
- new net: D1.2 (A), J2.1 (Pin_1)
- new net: LED_ESC_3.2 (A), R4.2
- new net SERVO_test: M1.1 (PWM), U2.37 (GPIO26)
Other:
- moved on the sheet: Cbst1, Cc1, Cc2, Cc3, Cin1, Cin10, Cin11, Cin12, Cin2, Cin3, Cin4, Cin5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

Commit message: 制御基板PCB7割完成
Parts:
- removed D1: SS34, Diode_SMD:D_SMA, symbol Diode:SS34
- removed D3, D4, D5, D6, D7: LED, LED_SMD:LED_0805_2012Metric, symbol Device:LED
- removed J1: Conn_01x02_Pin, Connector_PinHeader_2.54mm:PinHeader_1x02_P2.54mm_Vertical_SMD_Pin1Left, symbol Connector:Conn_01x02_Pin
- removed L1: 68u, Inductor_THT:L_Toroid_Vertical_L10.0mm_W5.0mm_P5.08mm, symbol Device:L
- removed R_tx0, R_tx1, R_tx2: 100k, Resistor_SMD:R_0603_1608Metric, symbol Device:R
- removed Y1: 8M, Crystal:Crystal_SMD_HC49-SD, symbol Device:Crystal
- added Analog_IN1: Conn_01x04_Pin, Connector_JST:JST_XH_B4B-XH-AM_1x04_P2.50mm_Vertical, symbol Connector:Conn_01x04_Pin
- added C1: 0.01u, Capacitor_SMD:C_0603_1608Metric, symbol Device:C
- added C4, C5: 100n, Capacitor_SMD:C_0603_1608Metric, symbol Device:C
- added CAN1: Conn_01x02_Pin, Connector_JST:JST_XH_B2B-XH-A_1x02_P2.50mm_Vertical, symbol Connector:Conn_01x02_Pin
- added CAN2: Conn_01x02_Pin, Connector_PinHeader_2.54mm:PinHeader_1x02_P2.54mm_Vertical, symbol Connector:Conn_01x02_Pin
- added D2: ~, basic_parts:SMA_L4.4-W2.8-LS5.4-R-RD, symbol basic_parts:SS54_C22452
- added H5, H6: MountingHole, MountingHole:MountingHole_3.2mm_M3, symbol Mechanical:MountingHole
- added J3: Conn_01x05_Pin, Connector_JST_additonal:JST_XA_S05B-XASK-1_1x05_P2.50mm_Horizontal, symbol Connector:Conn_01x05_Pin
- added J9: Barrel_Jack_Switch, Connector_BarrelJack:BarrelJack_Horizontal, symbol Connector:Barrel_Jack_Switch
- added JP2, JP3: SolderJumper_2_Open, Jumper:SolderJumper-2_P1.3mm_Open_RoundedPad1.0x1.5mm, symbol Jumper:SolderJumper_2_Open
- added L3: 10u, basic_parts:IND-SMD_L13.8-W12.6, symbol Device:L
- added M2: Fan, Connector_PinHeader_2.54mm:PinHeader_1x02_P2.54mm_Vertical, symbol Motor:Fan
- added TP2, TP4: TestPoint, Connector_Pin:Pin_D0.7mm_L6.5mm_W1.8mm_FlatFork, symbol Connector:TestPoint
- added U4: ADS1015IDGS, Package_SO:TSSOP-10_3x3mm_P0.5mm, symbol Analog_ADC:ADS1015IDGS
- added X1: 16MHz, basic_parts:OSC-SMD_4P-L3.2-W2.5-BL, symbol basic_parts:X322516MLB4SI
- Cc1, Cc2, Cc3: footprint Capacitor_SMD:C_0603_1608Metric -> Capacitor_SMD:C_0603_1608Metric_Pad1.08x0.95mm_HandSolder
- Cout2: value 0.1u -> 100p
- J4: value Conn_01x04_Pin -> SERVO_PWM
- R10: value 0.1 -> 100m; footprint Resistor_SMD:R_0201_0603Metric -> Resistor_SMD:R_1206_3216Metric; LCSC (none) -> C25334
- R12, R13: footprint Resistor_SMD:R_0201_0603Metric -> Resistor_SMD:R_0603_1608Metric
- R6, R7: value 200 -> 10k; footprint Resistor_SMD:R_0201_0603Metric -> Resistor_SMD:R_0603_1608Metric
- R8, R9: value 200 -> 5.1k; footprint Resistor_SMD:R_0201_0603Metric -> Resistor_SMD:R_0603_1608Metric
- R_CAN1: footprint Resistor_SMD:R_0603_1608Metric -> Resistor_SMD:R_1206_3216Metric; LCSC (none) -> C17909
- renumbered LED_ESC_5 to LED1, R_tx3 to R_reset1
Connections:
- net +5V is gone; now on net +5.1V: M1.2 (+), R10.1, R12.1, U1.5 (VIN), U2.2 (5V), U2.4 (5V), U3.3 (VCC)
- net +3.3V: now also Rpg1.2, C1.1, C4.2, J3.1 (Pin_1), JP2.1 (A), JP3.1 (A), U4.8 (VDD); no longer R6.1, R8.1, R9.1
- net +5.1V: now also C5.2, M2.1 (+), TP4.1
- net +7.5V: no longer Rpg1.2
- net BATTERY_OK: now also U2.18 (GPIO24); no longer U2.36 (GPIO16)
- net BLDC1_RP4: now also U2.40 (GPIO21(PCM_DOUT)); no longer U2.7 (GPIO4)
- net BLDC2_RP4: now also U2.35 (GPIO19(PCM_FS,_PWM1)); no longer U2.11 (GPIO17)
- net BLDC3_RP4: now also U2.36 (GPIO16); no longer U2.13 (GPIO27)
- net BLDC4_RP4: now also U2.32 (GPIO12(PWM0)); no longer U2.15 (GPIO22)
- net GND: now also R6.2, C1.2, C4.1, C5.1, J9.2, J9.3, M2.2 (-), TP2.1, U4.3 (GND), X1.4 (GND)
- net SERVO1: now also J4.4 (Pin_4), U2.33 (GPIO13(PWM1)); no longer J4.1 (Pin_1), U2.32 (GPIO12(PWM0))
- net SERVO2: now also J4.3 (Pin_3), U2.12 (GPIO18(PCM_CLK,_PWM0)); no longer J4.2 (Pin_2), U2.33 (GPIO13(PWM1))
- net SERVO3: now also J4.2 (Pin_2), U2.11 (GPIO17); no longer J4.3 (Pin_3), U2.16 (GPIO23)
- net SERVO4: now also J4.1 (Pin_1), U2.7 (GPIO4); no longer J4.4 (Pin_4), U2.18 (GPIO24)
- net at Q4.3 (D): now also J3.3 (Pin_3)
- net at R9.2: now also JP3.2 (B)
- net CANH: now reaches R_CAN1.1, U3.7 (CANH)
- net CANH: now also CAN1.1 (Pin_1), CAN2.1 (Pin_1)
- net at R1.1: now also D2.2 (K)
- net at R7.2: now also U4.2 (ALERT/RDY)
- net at R10.2, U1.4 (ISNS): now also J3.4 (Pin_4)
- net at U14.7 (OSC2): now also X1.2 (GND); no longer C2.2
- net CANL: now reaches JP1.1 (A), U3.6 (CANL)
- net CANL: now also CAN1.2 (Pin_2), CAN2.2 (Pin_2)
- net at Q3.3 (D): now also J3.2 (Pin_2)
- net at J2.1 (Pin_1): now also D2.1 (A), J9.1
- net at D8.2 (A), U1.1 (LX): now also L3.1
- net INT: now reaches U14.12 (~{INT})
- net INT: now also U2.38 (GPIO20(PCM_DIN))
- net at C3.2, U14.8 (OSC1): now also X1.1 (OSC1)
- net SDA: now reaches U15.3 (SDA), U2.3 (GPIO2(SDA))
- net SDA: now also R8.1, U4.9 (SDA)
- net SCL: now reaches U15.4 (SCL), U2.5 (GPIO3(SCL))
- net SCL: now also R9.1, U4.10 (SCL)
- net at R8.2: now also JP2.2 (B)
- net CS renamed CS0
- new net: R6.1, U4.1 (ADDR)
- new net: Analog_IN1.1 (Pin_1), U4.4 (AIN0)
- new net: Analog_IN1.2 (Pin_2), U4.5 (AIN1)
- new net: Analog_IN1.3 (Pin_3), U4.6 (AIN2)
- new net: Analog_IN1.4 (Pin_4), U4.7 (AIN3)
- new net: J3.5 (Pin_5), L3.2
- new net: C2.2, X1.3 (OSC2)
- no-connect marks 3 -> 14
Other:
- note added: "I2C Device"
- note added: "fsw = 40kHzくらい"
- note removed: "Low Power LED"
- moved on the sheet: C2, C3, H1, H2, H3, H4, J4, JP1, LED_BNO1, M1, Q3, R15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
