File: control_unit/control_unit.kicad_pcb (KiCad board)
At the start: 2 copper layers, 100 x 100 mm, 56 parts, among them J1 Conn_01x02_Pin, J2 Conn_01x02_Pin, J3 Conn_01x04_Pin, J4 Conn_01x04_Pin, J5 BLDC1, J6 Conn_01x04_Pin, J7 BLDC2, J8 BLDC3, J9 BLDC4, Q1 AO3401A, Q2 2N7002, U4 BNO055, U5 OKL-T/6-W12N-C

Commit message: OKL[200~過渡応答を
Parts:
- removed C10, C3, C4, C5, C6, C7, C8, C9: 22uF, Capacitor_SMD:C_1206_3216Metric
- removed D2: LED, LED_SMD:LED_0805_2012Metric
- removed D9: SS34, Diode_SMD:D_SMA
- removed J2: Conn_01x02_Pin, Connector_PinHeader_2.54mm:PinHeader_1x02_P2.54mm_Vertical
- removed J3, J6: Conn_01x04_Pin, Connector_PinHeader_2.54mm:PinHeader_1x04_P2.54mm_Vertical
- removed R1: 100k, Resistor_SMD:R_0201_0603Metric
- removed R2, R3: 20k, Resistor_SMD:R_0201_0603Metric
- removed R4: 100, Resistor_SMD:R_0201_0603Metric
- removed R5: 1.2k, Resistor_SMD:R_0201_0603Metric
- removed RV1: R_Potentiometer, basic_parts:RES-ADJ-SMD_GF063P1
- added Cin1: 10u, Capacitor_SMD:C_1210_3225Metric_Pad1.33x2.70mm_HandSolder, F.Cu at (55.0, 55.9)
- added Cin10: 10u, Capacitor_SMD:C_1210_3225Metric_Pad1.33x2.70mm_HandSolder, F.Cu at (61.0, 68.6)
- added Cin11: 10u, Capacitor_SMD:C_1210_3225Metric_Pad1.33x2.70mm_HandSolder, F.Cu at (61.0, 72.9)
- added Cin12: 10u, Capacitor_SMD:C_1210_3225Metric_Pad1.33x2.70mm_HandSolder, F.Cu at (61.0, 77.1)
- added Cin13: 10u, Capacitor_SMD:C_1210_3225Metric_Pad1.33x2.70mm_HandSolder, F.Cu at (67.0, 55.9)
- added Cin14: 10u, Capacitor_SMD:C_1210_3225Metric_Pad1.33x2.70mm_HandSolder, F.Cu at (67.0, 60.1)
- added Cin15: 10u, Capacitor_SMD:C_1210_3225Metric_Pad1.33x2.70mm_HandSolder, F.Cu at (67.0, 64.4)
- added Cin16: 10u, Capacitor_SMD:C_1210_3225Metric_Pad1.33x2.70mm_HandSolder, F.Cu at (67.0, 68.6)
- added Cin17: 10u, Capacitor_SMD:C_1210_3225Metric_Pad1.33x2.70mm_HandSolder, F.Cu at (67.0, 72.9)
- added Cin2: 10u, Capacitor_SMD:C_1210_3225Metric_Pad1.33x2.70mm_HandSolder, F.Cu at (55.0, 60.1)
- added Cin3: 10u, Capacitor_SMD:C_1210_3225Metric_Pad1.33x2.70mm_HandSolder, F.Cu at (55.0, 64.4)
- added Cin4: 10u, Capacitor_SMD:C_1210_3225Metric_Pad1.33x2.70mm_HandSolder, F.Cu at (55.0, 68.6)
- added Cin5: 10u, Capacitor_SMD:C_1210_3225Metric_Pad1.33x2.70mm_HandSolder, F.Cu at (55.0, 72.9)
- added Cin6: 10u, Capacitor_SMD:C_1210_3225Metric_Pad1.33x2.70mm_HandSolder, F.Cu at (55.0, 77.1)
- added Cin7: 10u, Capacitor_SMD:C_1210_3225Metric_Pad1.33x2.70mm_HandSolder, F.Cu at (61.0, 55.9)
- added Cin8: 10u, Capacitor_SMD:C_1210_3225Metric_Pad1.33x2.70mm_HandSolder, F.Cu at (61.0, 60.1)
- added Cin9: 10u, Capacitor_SMD:C_1210_3225Metric_Pad1.33x2.70mm_HandSolder, F.Cu at (61.0, 64.4)
- added Cout1: 47u, Capacitor_SMD:C_1210_3225Metric, F.Cu at (66.9, 81.4)
- added Cout2: 47u, Capacitor_SMD:C_1210_3225Metric, F.Cu at (66.9, 85.6)
- added Cout3: 47u, Capacitor_SMD:C_1210_3225Metric, F.Cu at (66.9, 89.9)
- added Cout4: 47u, Capacitor_SMD:C_1210_3225Metric, F.Cu at (66.9, 94.1)
- added H1: MountingHole, MountingHole:MountingHole_3.2mm_M3, F.Cu at (48.0, 57.7)
- added H2: MountingHole, MountingHole:MountingHole_3.2mm_M3, F.Cu at (48.0, 65.7)
- added H3: MountingHole, MountingHole:MountingHole_3.2mm_M3, F.Cu at (48.0, 73.6)
- added H4: MountingHole, MountingHole:MountingHole_3.2mm_M3, F.Cu at (48.0, 81.6)
- added Q2: ~, Package_TO_SOT_SMD:TO-252-2, F.Cu at (76.7, 91.6)
- added Q4: 2N7002, Package_TO_SOT_SMD:SOT-23, F.Cu at (79.0, 98.0)
- added U14: MCP2515-xSO, Package_SO:SOIC-18W_7.5x11.6mm_P1.27mm, F.Cu at (88.3, 85.9)
- added U15: BNO055 DIP, myfootprint:BNO055 DIP, F.Cu at (58.0, 88.8)
- Q1: value AO3401A -> ~; footprint Package_TO_SOT_SMD:SOT-23 -> Package_TO_SOT_SMD:TO-252-2
- U3: value ~ -> ATA6561-GAQW-N; footprint basic_parts:RES-ADJ-SMD_GF063P1 -> ATA6561:SOIC8_4P9X3P9MC_MCH
- U4: value BNO055 -> ~; footprint Package_LGA:LGA-28_5.2x3.8mm_P0.5mm -> basic_parts:wetness sensor
- U5: value OKL-T/6-W12N-C -> ~; footprint OKL-T6-W12N-C:OKL-T&slash_6-W12N-C_MUR -> basic_parts:VQFN-20_L4.5-W3.5-P0.50-BL-EP
- moved Q1 107.5 mm to (76.7, 83.4)
- moved U3 97.7 mm to (86.2, 95.7)
- moved U4 93.2 mm to (81.4, 75.2)
- moved U5 73.2 mm to (73.4, 98.3)
- moved U2 5.64 mm to (183.2, 122.5)
- renumbered Q2 to Q3
Connections:
- D4 pad 1: Net-(D3-K) -> Net-(D4-K)
- D6 pad 1: Net-(D3-K) -> Net-(D4-K)
- D8 pad 1: GND -> +24V
- J1 pad 2: GND -> +24V
- J5 pad 2: unconnected-(J5-Pin_2-Pad2) -> Net-(J5-Pin_2)
- J5 pad 3: GND -> +24V
- J7 pad 2: unconnected-(J7-Pin_2-Pad2) -> Net-(J7-Pin_2)
- J7 pad 3: GND -> +24V
- J8 pad 2: unconnected-(J8-Pin_2-Pad2) -> Net-(J8-Pin_2)
- J8 pad 3: GND -> +24V
- J9 pad 2: unconnected-(J9-Pin_2-Pad2) -> Net-(J9-Pin_2)
- J9 pad 3: GND -> +24V
- Q1 pad 2: Net-(Q1-S) -> +24V
- Q1 pad 3: +5V -> Net-(Q1-S)
- Q3 pad 2: GND -> +24V
- R13 pad 2: GND -> +24V
- U1 pad 2: GND -> +24V
- U10 pad 1: GND -> +24V
- U10 pad 2: SERVO_LOGIC -> +5V
- U10 pad 4: GND -> +24V
- U11 pad 1: GND -> +24V
- U11 pad 2: SERVO_LOGIC -> +5V
- U11 pad 4: GND -> +24V
- U12 pad 1: GND -> +24V
- U12 pad 2: SERVO_LOGIC -> +5V
- U12 pad 4: GND -> +24V
- U13 pad 1: GND -> +24V
- U13 pad 2: SERVO_LOGIC -> +5V
- U13 pad 4: GND -> +24V
- U2 pad 14: GND -> +24V
- U2 pad 19: unconnected-(U2-GPIO10(MOSI)-Pad19) -> MOSI
- U2 pad 20: GND -> +24V
- U2 pad 21: LowBeam -> MISO
- U2 pad 22: unconnected-(U2-GPIO25-Pad22) -> IR
- U2 pad 23: unconnected-(U2-GPIO11(SCLK)-Pad23) -> SCK
- U2 pad 24: unconnected-(U2-GPIO8(CE0)-Pad24) -> CS
- U2 pad 25: GND -> +24V
- U2 pad 3: Net-(U2-GPIO2(SDA)) -> Net-(U15-SDA)
- U2 pad 30: GND -> +24V
- U2 pad 31: unconnected-(U2-GPIO6-Pad31) -> LowBeam
- U2 pad 34: GND -> +24V
- U2 pad 36: unconnected-(U2-GPIO16-Pad36) -> BATTERY_OK
- U2 pad 37: unconnected-(U2-GPIO26-Pad37) -> Net-(U2-GPIO26)
- U2 pad 39: GND -> +24V
- U2 pad 5: Net-(U2-GPIO3(SCL)) -> Net-(U15-SCL)
- U2 pad 6: GND -> +24V
- U2 pad 9: GND -> +24V
- U3 pad 1: Net-(U2-GPIO3(SCL)) -> Net-(U14-TXCAN)
- U3 pad 2: Net-(U2-GPIO2(SDA)) -> +24V
- U3 pad 3: +3.3V -> +5V
- U4 pad 1: unconnected-(U4-PIN1-Pad1) -> Net-(U2-GPIO26)
- U4 pad 2: GND -> +24V
- U5 pad 10: Net-(U5-PG) -> PGOOD
- U5 pad 11: unconnected-(U5-NC-Pad11) -> Net-(U5-ILIM)
- U5 pad 12: unconnected-(U5-NC-Pad12) -> +24V
- U5 pad 2: VCC -> Net-(U5-RT)
- U5 pad 3: GND -> Net-(U5-SS/TRK)
- U5 pad 4: +5V -> Net-(U5-COMP)
- U5 pad 5: +5V -> Net-(U5-FB)
- U5 pad 6: Net-(U5-TRIM1) -> +24V
- U5 pad 7: GND -> unconnected-(U5-SYNCOUT-Pad7)
- U5 pad 8: unconnected-(U5-NC-Pad8) -> +24V
- U6 pad 1: GND -> +24V
- U6 pad 4: GND -> +24V
- U7 pad 1: GND -> +24V
- U7 pad 4: GND -> +24V
- U8 pad 1: GND -> +24V
- U8 pad 4: GND -> +24V
- U9 pad 1: GND -> +24V
- U9 pad 4: GND -> +24V
Other:
- board size 100 x 100 mm -> 2 x 17 mm

Commit message: 制御基板配線開始
Parts:
- removed Cin13, Cin14, Cin15, Cin16, Cin17: 10u, Capacitor_SMD:C_1210_3225Metric_Pad1.33x2.70mm_HandSolder
- removed J9: BLDC4, Connector_PinHeader_2.54mm:PinHeader_1x03_P2.54mm_Vertical
- removed U10, U11, U12, U13, U6, U7, U8, U9: ~, basic_parts:SOT-23-5_L3.0-W1.7-P0.95-LS2.8-BR
- removed U4: ~, basic_parts:wetness sensor
- added C2: 22p, Capacitor_SMD:C_0603_1608Metric, F.Cu at (83.5, 22.0)
- added C3: 22p, Capacitor_SMD:C_0603_1608Metric, F.Cu at (83.5, 24.6)
- added Cbst1: 0.1u, Capacitor_SMD:C_0603_1608Metric, F.Cu at (83.5, 27.1)
- added Cc1: 5.6n, Capacitor_SMD:C_0603_1608Metric, F.Cu at (83.5, 29.6)
- added Cc2: 82p, Capacitor_SMD:C_0603_1608Metric, F.Cu at (83.5, 32.1)
- added Cc3: 1500p, Capacitor_SMD:C_0603_1608Metric, F.Cu at (83.5, 34.6)
- added Cout1: 100p, Capacitor_SMD:C_0603_1608Metric, F.Cu at (83.5, 37.1)
- added Cout2: 0.1u, Capacitor_SMD:C_0603_1608Metric, F.Cu at (87.5, 22.0)
- added Cout3: 47u, Capacitor_SMD:C_1210_3225Metric, F.Cu at (112.1, 57.4)
- added Css1: 0.1u, Capacitor_SMD:C_0603_1608Metric, F.Cu at (87.5, 24.6)
- added Cvcc1: 2.2u, Capacitor_SMD:C_0603_1608Metric, F.Cu at (87.5, 27.1)
- added Cvin1: 0.1u, Capacitor_SMD:C_0603_1608Metric, F.Cu at (87.5, 29.6)
- added J2: Conn_01x02_Socket, Connector_JST:JST_VH_B2P-VH_1x02_P3.96mm_Vertical, B.Cu at (153.0, 49.0)
- added J6: BLDC1, Connector_PinHeader_2.54mm:PinHeader_1x03_P2.54mm_Vertical, F.Cu at (99.8, 37.4)
- added JP1: Jumper_2_Bridged, TestPoint:TestPoint_2Pads_Pitch2.54mm_Drill0.8mm, F.Cu at (114.0, 46.4)
- added L2: 10u, basic_parts:IND-SMD_L13.8-W12.6, F.Cu at (213.2, 47.0)
- added LED_BNO1: GREEN, LED_SMD:LED_1206_3216Metric, F.Cu at (84.3, 40.0)
- added LED_ESC_1: GREEN, LED_SMD:LED_1206_3216Metric, F.Cu at (84.3, 43.4)
- added LED_ESC_2: GREEN, LED_SMD:LED_1206_3216Metric, F.Cu at (84.3, 46.8)
- added LED_ESC_3: GREEN, LED_SMD:LED_1206_3216Metric, F.Cu at (84.3, 50.2)
- added LED_ESC_4: GREEN, LED_SMD:LED_1206_3216Metric, F.Cu at (84.3, 53.6)
- added LED_ESC_5: GREEN, LED_SMD:LED_1206_3216Metric, F.Cu at (84.3, 57.0)
- added M1: Motor_Servo, Connector_PinHeader_2.54mm:PinHeader_1x03_P2.54mm_Vertical, F.Cu at (113.8, 37.4)
- added R1: 20m, Diode_SMD:D_2010_5025Metric_Pad1.52x2.65mm_HandSolder, F.Cu at (162.0, 48.0)
- added R14: 1.2k, Resistor_SMD:R_0603_1608Metric, F.Cu at (91.5, 24.6)
- added R15: 1.2k, Resistor_SMD:R_0603_1608Metric, F.Cu at (91.5, 27.1)
- added R2: 1.2k, Resistor_SMD:R_0603_1608Metric, F.Cu at (87.5, 32.1)
- added R3: 1.2k, Resistor_SMD:R_0603_1608Metric, F.Cu at (87.5, 34.6)
- added R4: 1.2k, Resistor_SMD:R_0603_1608Metric, F.Cu at (87.5, 37.1)
- added R5: 1.2k, Resistor_SMD:R_0603_1608Metric, F.Cu at (91.5, 22.0)
- added R_CAN1: 120, Resistor_SMD:R_0603_1608Metric, F.Cu at (91.5, 29.6)
- added R_tx0: 100k, Resistor_SMD:R_0603_1608Metric, F.Cu at (91.5, 32.1)
- added R_tx1: 100k, Resistor_SMD:R_0603_1608Metric, F.Cu at (91.5, 34.6)
- added R_tx2: 100k, Resistor_SMD:R_0603_1608Metric, F.Cu at (91.5, 37.1)
- added R_tx3: 100k, Resistor_SMD:R_0603_1608Metric, F.Cu at (95.5, 22.0)
- added Rc1: 10k, Resistor_SMD:R_0603_1608Metric_Pad0.98x0.95mm_HandSolder, F.Cu at (89.3, 50.2)
- added Rc2: 560, Resistor_SMD:R_0603_1608Metric_Pad0.98x0.95mm_HandSolder, F.Cu at (89.3, 52.7)
- added Rfb1: 18k, Resistor_SMD:R_0603_1608Metric_Pad0.98x0.95mm_HandSolder, F.Cu at (89.3, 55.2)
- added Rfb2: 3.3k, Resistor_SMD:R_0603_1608Metric_Pad0.98x0.95mm_HandSolder, F.Cu at (89.3, 57.7)
- added Rilim1: 180, Resistor_SMD:R_0603_1608Metric, F.Cu at (95.5, 24.6)
- added Rpg1: 51k, Resistor_SMD:R_0603_1608Metric, F.Cu at (95.5, 27.1)
- added Rt1: 33k, Resistor_SMD:R_0603_1608Metric, F.Cu at (95.5, 29.6)
- added Ruv1: 75k, Resistor_SMD:R_0603_1608Metric, F.Cu at (95.5, 32.1)
- added Ruv2: 12k, Resistor_SMD:R_0603_1608Metric, F.Cu at (95.5, 34.6)
- added TP1: TestPoint, Connector_Pin:Pin_D0.7mm_L6.5mm_W1.8mm_FlatFork, F.Cu at (117.0, 57.0)
- added Y1: 8M, Crystal:Crystal_SMD_HC49-SD, F.Cu at (104.8, 47.9)
- Cin1, Cin10, Cin11, Cin12, Cin2, Cin3, Cin4, Cin5, Cin6, Cin7, Cin8, Cin9: footprint Capacitor_SMD:C_1210_3225Metric_Pad1.33x2.70mm_HandSolder -> Capacitor_SMD:C_1210_3225Metric
- J4: footprint Connector_PinHeader_2.54mm:PinHeader_1x04_P2.54mm_Vertical -> Connector_JST:JST_XH_B4B-XH-A_1x04_P2.50mm_Vertical
- J7: value BLDC2 -> BLDC1
- J8: value BLDC3 -> BLDC1
- moved Q3 303.4 mm to (429.2, -24.3), turned to 90 degrees
- moved J1 296.7 mm to (425.7, -30.7), turned to 90 degrees
- moved D8 293.5 mm to (420.3, -17.8), turned to 90 degrees
- moved R8 286.6 mm to (419.6, -37.1), turned to 90 degrees
- moved R13 286.0 mm to (419.6, -39.5), turned to 90 degrees
- moved R7 284.2 mm to (417.9, -37.1), turned to 90 degrees
- moved R12 283.6 mm to (417.9, -39.5), turned to 90 degrees
- moved L1 283.2 mm to (415.3, -27.6), turned to 90 degrees
- moved R6 281.7 mm to (416.1, -37.1), turned to 90 degrees
- moved R10 281.1 mm to (416.1, -39.5), turned to 90 degrees
- moved R9 278.7 mm to (414.4, -39.5), turned to 90 degrees
- moved U1 273.0 mm to (409.3, -34.2), turned to 90 degrees
- moved R11 238.5 mm to (384.6, -35.0), turned to 90 degrees
- moved D7 219.5 mm to (371.6, -38.8), turned to 90 degrees
- moved D6 215.3 mm to (368.6, -38.8), turned to 90 degrees
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- renumbered Cout1 to Cout4, Cout2 to Cout5, Cout3 to Cout6, Cout4 to Cout7
Connections:
- Cin1 pad 2: +24V -> GND
- Cin10 pad 2: +24V -> GND
- Cin11 pad 2: +24V -> GND
- Cin12 pad 2: +24V -> GND
- Cin2 pad 2: +24V -> GND
- Cin3 pad 2: +24V -> GND
- Cin4 pad 2: +24V -> GND
- Cin5 pad 2: +24V -> GND
- Cin6 pad 2: +24V -> GND
- Cin7 pad 2: +24V -> GND
- Cin8 pad 2: +24V -> GND
- Cin9 pad 2: +24V -> GND
- Cout4 pad 2: +24V -> GND
- Cout5 pad 2: +24V -> GND
- Cout6 pad 2: +24V -> GND
- Cout7 pad 2: +24V -> GND
- D1 pad 1: SERVO_LOGIC -> Net-(D1-K)
- D1 pad 2: +5V -> Net-(D1-A)
- D8 pad 1: +24V -> GND
- J1 pad 2: +24V -> GND
- J4 pad 1: Net-(J4-Pin_1) -> SERVO1
- J4 pad 2: Net-(J4-Pin_2) -> SERVO2
- J4 pad 3: Net-(J4-Pin_3) -> SERVO3
- J4 pad 4: Net-(J4-Pin_4) -> SERVO4
- J5 pad 1: Net-(J5-Pin_1) -> BLDC1_RP4
- J5 pad 3: +24V -> GND
- J7 pad 1: Net-(J7-Pin_1) -> BLDC3_RP4
- J7 pad 3: +24V -> GND
- J8 pad 1: Net-(J8-Pin_1) -> BLDC4_RP4
- J8 pad 3: +24V -> GND
- Q2 pad 3: +24V -> GND
- Q3 pad 2: +24V -> GND
- Q4 pad 2: +24V -> GND
- R13 pad 2: +24V -> GND
- U1 pad 2: +24V -> GND
- U14 pad 9: +24V -> GND
- U15 pad 2: +24V -> GND
- U15 pad 7: +24V -> GND
- U2 pad 14: +24V -> GND
- U2 pad 16: Net-(U2-GPIO23) -> SERVO3
- U2 pad 18: Net-(U2-GPIO24) -> SERVO4
- U2 pad 20: +24V -> GND
- U2 pad 25: +24V -> GND
- U2 pad 30: +24V -> GND
- U2 pad 32: Net-(U2-GPIO12(PWM0)) -> SERVO1
- U2 pad 33: Net-(U2-GPIO13(PWM1)) -> SERVO2
- U2 pad 34: +24V -> GND
- U2 pad 37: Net-(U2-GPIO26) -> SERVO_test
- U2 pad 39: +24V -> GND
- U2 pad 6: +24V -> GND
- U2 pad 9: +24V -> GND
- U3 pad 2: +24V -> GND
- U3 pad 8: +24V -> GND
- U5 pad 12: +24V -> GND
- U5 pad 15: +24V -> GND
- U5 pad 16: +24V -> GND
- U5 pad 21: +24V -> GND
- U5 pad 6: +24V -> GND
- U5 pad 8: +24V -> GND
Other:
- board size 2 x 17 mm -> 100 x 95 mm

Commit message: 制御基板PCB7割完成
Parts:
- removed D1: SS34, Diode_SMD:D_SMA
- removed D3, D4, D5, D6, D7: LED, LED_SMD:LED_0805_2012Metric
- removed J1: Conn_01x02_Pin, Connector_PinHeader_2.54mm:PinHeader_1x02_P2.54mm_Vertical_SMD_Pin1Left
- removed L1: 68u, Inductor_THT:L_Toroid_Vertical_L10.0mm_W5.0mm_P5.08mm
- removed LED_ESC_5: GREEN, LED_SMD:LED_1206_3216Metric
- removed R_tx0, R_tx1, R_tx2, R_tx3: 100k, Resistor_SMD:R_0603_1608Metric
- removed Y1: 8M, Crystal:Crystal_SMD_HC49-SD
- added Analog_IN1: Conn_01x04_Pin, Connector_JST:JST_XH_B4B-XH-AM_1x04_P2.50mm_Vertical, B.Cu at (145.5, 45.5)
- added C1: 0.01u, Capacitor_SMD:C_0603_1608Metric, F.Cu at (158.0, 53.0)
- added C4: 100n, Capacitor_SMD:C_0603_1608Metric, F.Cu at (200.0, 70.5)
- added C5: 100n, Capacitor_SMD:C_0603_1608Metric, F.Cu at (197.6, 66.6)
- added CAN1: Conn_01x02_Pin, Connector_JST:JST_XH_B2B-XH-A_1x02_P2.50mm_Vertical, B.Cu at (145.5, 73.5)
- added CAN2: Conn_01x02_Pin, Connector_PinHeader_2.54mm:PinHeader_1x02_P2.54mm_Vertical, F.Cu at (151.8, 73.5)
- added D2: ~, basic_parts:SMA_L4.4-W2.8-LS5.4-R-RD, F.Cu at (146.8, 106.5)
- added H5: MountingHole, MountingHole:MountingHole_3.2mm_M3, F.Cu at (236.0, 51.5)
- added H6: MountingHole, MountingHole:MountingHole_3.2mm_M3, F.Cu at (236.0, 101.5)
- added J3: Conn_01x05_Pin, Connector_JST_additonal:JST_XA_S05B-XASK-1_1x05_P2.50mm_Horizontal, F.Cu at (268.5, 92.0)
- added J9: Barrel_Jack_Switch, Connector_BarrelJack:BarrelJack_Horizontal, F.Cu at (155.0, 84.0)
- added JP2: SolderJumper_2_Open, Jumper:SolderJumper-2_P1.3mm_Open_RoundedPad1.0x1.5mm, F.Cu at (200.0, 77.8)
- added JP3: SolderJumper_2_Open, Jumper:SolderJumper-2_P1.3mm_Open_RoundedPad1.0x1.5mm, F.Cu at (200.0, 75.0)
- added L3: 10u, basic_parts:IND-SMD_L13.8-W12.6, F.Cu at (227.5, 93.8)
- added LED1: GREEN, LED_SMD:LED_1206_3216Metric, F.Cu at (174.0, 41.5)
- added M2: Fan, Connector_PinHeader_2.54mm:PinHeader_1x02_P2.54mm_Vertical, F.Cu at (160.5, 84.5)
- added R_reset1: 100k, Resistor_SMD:R_0603_1608Metric, F.Cu at (199.0, 50.2)
- added TP2: TestPoint, Connector_Pin:Pin_D0.7mm_L6.5mm_W1.8mm_FlatFork, F.Cu at (146.5, 110.8)
- added TP4: TestPoint, Connector_Pin:Pin_D0.7mm_L6.5mm_W1.8mm_FlatFork, F.Cu at (190.5, 97.8)
- added U4: ADS1015IDGS, Package_SO:TSSOP-10_3x3mm_P0.5mm, F.Cu at (153.0, 52.8)
- added X1: 16MHz, basic_parts:OSC-SMD_4P-L3.2-W2.5-BL, F.Cu at (212.2, 56.9)
- Cc1, Cc2, Cc3: footprint Capacitor_SMD:C_0603_1608Metric -> Capacitor_SMD:C_0603_1608Metric_Pad1.08x0.95mm_HandSolder
- Cout2: value 0.1u -> 100p
- J4: value Conn_01x04_Pin -> SERVO_PWM; moved to B.Cu
- R10: value 0.1 -> 100m; footprint Resistor_SMD:R_0201_0603Metric -> Resistor_SMD:R_1206_3216Metric
- R12, R13: footprint Resistor_SMD:R_0201_0603Metric -> Resistor_SMD:R_0603_1608Metric
- R6, R7: value 200 -> 10k; footprint Resistor_SMD:R_0201_0603Metric -> Resistor_SMD:R_0603_1608Metric
- R8, R9: value 200 -> 5.1k; footprint Resistor_SMD:R_0201_0603Metric -> Resistor_SMD:R_0603_1608Metric
- R_CAN1: footprint Resistor_SMD:R_0603_1608Metric -> Resistor_SMD:R_1206_3216Metric
- moved R7 280.7 mm to (153.0, 55.8), turned to 180 degrees
- moved R6 278.3 mm to (151.8, 50.0), turned to 0 degrees
- moved R8 243.7 mm to (204.5, 77.5), turned to 180 degrees
- moved R9 239.1 mm to (204.5, 75.0), turned to 180 degrees
- moved R12 207.1 mm to (253.7, 86.8), turned to 0 degrees
- moved Q3 204.5 mm to (260.9, 92.0), turned to 0 degrees
- moved R13 202.7 mm to (253.9, 77.2), turned to 180 degrees
- moved H4 193.9 mm to (236.0, 34.0)
- moved H3 193.4 mm to (236.0, 119.0)
- moved R10 189.5 mm to (266.9, 77.2), turned to 0 degrees
- moved D8 187.9 mm to (262.4, 84.0), turned to 180 degrees
- moved U1 186.0 mm to (261.6, 78.9)
- moved Q4 182.1 mm to (260.9, 88.0)
- moved R11 174.9 mm to (254.3, 81.8)
- moved U15 151.9 mm to (209.4, 76.3), turned to -90 degrees
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Connections:
- net CS renamed CS0
- net Net-(JP1-A) renamed CANL
- net Net-(U3-CANH) renamed CANH
- C2 pad 2: Net-(U14-OSC2) -> Net-(X1-OSC2)
- J4 pad 1: SERVO1 -> SERVO4
- J4 pad 2: SERVO2 -> SERVO3
- J4 pad 3: SERVO3 -> SERVO2
- J4 pad 4: SERVO4 -> SERVO1
- M1 pad 2: +5V -> +5.1V
- R10 pad 1: +5V -> +5.1V
- R12 pad 1: +5V -> +5.1V
- R6 pad 1: +3.3V -> Net-(U4-ADDR)
- R6 pad 2: Net-(D5-A) -> GND
- R8 pad 1: +3.3V -> SDA
- R9 pad 1: +3.3V -> SCL
- Rpg1 pad 2: +7.5V -> +3.3V
- U1 pad 5: +5V -> +5.1V
- U14 pad 12: unconnected-(U14-~{INT}-Pad12) -> INT
- U14 pad 4: Net-(U14-~{TX0RTS}) -> unconnected-(U14-~{TX0RTS}-Pad4)
- U14 pad 5: Net-(U14-~{TX1RTS}) -> unconnected-(U14-~{TX1RTS}-Pad5)
- U14 pad 6: Net-(U14-~{TX2RTS}) -> unconnected-(U14-~{TX2RTS}-Pad6)
- U15 pad 3: Net-(U15-SDA) -> SDA
- U15 pad 4: Net-(U15-SCL) -> SCL
- U2 pad 11: BLDC2_RP4 -> SERVO3
- U2 pad 12: unconnected-(U2-GPIO18(PCM_CLK)-Pad12) -> SERVO2
- U2 pad 13: BLDC3_RP4 -> unconnected-(U2-GPIO27-Pad13)
- U2 pad 15: BLDC4_RP4 -> unconnected-(U2-GPIO22-Pad15)
- U2 pad 16: SERVO3 -> unconnected-(U2-GPIO23-Pad16)
- U2 pad 18: SERVO4 -> BATTERY_OK
- U2 pad 2: +5V -> +5.1V
- U2 pad 3: Net-(U15-SDA) -> SDA
- U2 pad 32: SERVO1 -> BLDC4_RP4
- U2 pad 33: SERVO2 -> SERVO1
- U2 pad 35: unconnected-(U2-GPIO19(PCM_FS)-Pad35) -> BLDC2_RP4
- U2 pad 36: BATTERY_OK -> BLDC3_RP4
- U2 pad 38: unconnected-(U2-GPIO20(PCM_DIN)-Pad38) -> INT
- U2 pad 4: +5V -> +5.1V
- U2 pad 40: unconnected-(U2-GPIO21(PCM_DOUT)-Pad40) -> BLDC1_RP4
- U2 pad 5: Net-(U15-SCL) -> SCL
- U2 pad 7: BLDC1_RP4 -> SERVO4
- U3 pad 3: +5V -> +5.1V
- U5 pad 9: unconnected-(U5-NC-Pad9) -> GND
Routing:
- net +5.1V: track 0.00 -> 97.1 mm, vias 0 -> 2
- net SDA: track 0.00 -> 83.2 mm, vias 0 -> 3
- net SCL: track 0.00 -> 77.0 mm, vias 0 -> 3
- net CANH: track 0.00 -> 75.0 mm, vias 0 -> 2
- net CANL: track 0.00 -> 74.0 mm, vias 0 -> 2
- net +3.3V: track 0.00 -> 72.5 mm, vias 0 -> 2
- net SERVO1: track 0.00 -> 67.8 mm
- net SERVO2: track 0.00 -> 38.9 mm
- net BLDC4_RP4: track 0.00 -> 37.4 mm
- net SERVO3: track 0.00 -> 33.6 mm
- net Net-(D2-A): track 0.00 -> 29.3 mm
- net MOSI: track 0.00 -> 28.6 mm
- net SERVO4: track 0.00 -> 28.4 mm
- net +24V: track 0.00 -> 28.2 mm, vias 0 -> 3
- net BLDC3_RP4: track 0.00 -> 27.1 mm
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- added copper zone on F.Cu, net +24V
- added copper zone on F.Cu, net +5.1V
- added copper zone on F.Cu, net GND
- added copper zone on F.Cu, net Net-(Q1-S)
Other:
- board text added: "HEAT SINK AREA"

Commit message: 配線完了
Parts:
- removed J3: Conn_01x05_Pin, Connector_JST_additonal:JST_XA_S05B-XASK-1_1x05_P2.50mm_Horizontal
- added J1: Conn_02x03_Counter_Clockwise, Connector_PinHeader_2.54mm:PinHeader_2x03_P2.54mm_Vertical, F.Cu at (142.3, 132.3)
- added Q7: AO3400A, Package_TO_SOT_SMD:SOT-23, F.Cu at (138.3, 73.6)
- added Q8: AO3400A, Package_TO_SOT_SMD:SOT-23, F.Cu at (138.3, 79.6)
- added R17: 10k, Resistor_SMD:R_0603_1608Metric, F.Cu at (137.3, 95.3)
- added R18: 10k, Resistor_SMD:R_0603_1608Metric, F.Cu at (138.1, 70.9)
- added R19: 10k, Resistor_SMD:R_0603_1608Metric, F.Cu at (144.0, 88.8)
- added R20: 100k, Resistor_SMD:R_0603_1608Metric, F.Cu at (144.1, 92.6)
- added R21: 10k, Resistor_SMD:R_0603_1608Metric, F.Cu at (138.1, 76.9)
- Q4: value 2N7002 -> MMBT5551L
- moved R10 133.7 mm to (143.5, 128.8)
- moved U1 127.1 mm to (143.2, 124.8), turned to 180 degrees
- moved R2 126.2 mm to (123.5, 136.1)
- moved J5 125.9 mm to (125.0, 127.6)
- moved R3 125.8 mm to (127.8, 136.1)
- moved J6 125.5 mm to (129.3, 127.6)
- moved R4 125.4 mm to (132.2, 136.2)
- moved J7 125.2 mm to (133.5, 127.6)
- moved D8 125.1 mm to (142.8, 120.6), turned to 0 degrees
- moved R5 124.9 mm to (136.5, 136.3)
- moved J8 124.4 mm to (138.0, 127.6)
- moved LED_ESC_1 122.0 mm to (125.8, 137.1)
- moved LED_ESC_2 121.6 mm to (130.0, 137.1)
- moved R11 121.4 mm to (133.3, 90.8)
- moved LED_ESC_3 121.2 mm to (134.4, 137.2)
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Connections:
- C1 pad 1: +3.3V -> +3.3V_1
- C2 pad 2: Net-(X1-OSC2) -> Net-(U14-OSC2)
- C4 pad 2: +3.3V -> +3.3V_2
- D8 pad 1: GND -> +5.1V
- JP2 pad 1: +3.3V -> +3.3V_2
- JP3 pad 1: +3.3V -> +3.3V_2
- Q3 pad 1: LowBeam -> Net-(Q3-G)
- Q3 pad 3: Net-(J3-Pin_2) -> Net-(Q3-D)
- Q4 pad 1: IR -> Net-(Q4-B)
- Q4 pad 3: Net-(J3-Pin_3) -> Net-(Q3-G)
- R11 pad 2: HighBeam -> Net-(Q3-D)
- R7 pad 1: +3.3V -> +3.3V_1
- R_reset1 pad 2: +3.3V -> +3.3V_2
- Rpg1 pad 2: +3.3V -> +3.3V_2
- U1 pad 3: (no net) -> Net-(Q3-D)
- U14 pad 18: +3.3V -> +3.3V_2
- U15 pad 1: +3.3V -> +3.3V_2
- U2 pad 1: +3.3V -> +3.3V_1
- U2 pad 17: +3.3V -> +3.3V_2
- U3 pad 5: +3.3V -> +3.3V_2
- U4 pad 8: +3.3V -> +3.3V_1
- X1 pad 2: Net-(U14-OSC2) -> GND
- X1 pad 3: Net-(X1-OSC2) -> Net-(U14-OSC2)
Routing:
- net +5.1V: track 97.1 -> 216.1 mm, vias 2 -> 16
- net +3.3V_2: track 0.00 -> 85.1 mm, vias 0 -> 5
- net +3.3V: track 72.5 -> 0.00 mm, vias 2 -> 0
- net Net-(J1-Pin_3): track 0.00 -> 67.8 mm, vias 0 -> 1
- net Net-(J1-Pin_2): track 0.00 -> 67.7 mm, vias 0 -> 1
- net BLDC4_RP4: track 37.4 -> 98.3 mm
- net BLDC3_RP4: track 27.1 -> 87.2 mm
- net BLDC2_RP4: track 25.1 -> 84.2 mm
- net SERVO_test: track 0.00 -> 55.9 mm, vias 0 -> 3
- net BLDC1_RP4: track 17.6 -> 72.9 mm
- net Net-(Q3-D): track 0.00 -> 47.3 mm, vias 0 -> 5
- net IR: track 0.00 -> 42.9 mm, vias 0 -> 4
- net HighBeam: track 0.00 -> 42.7 mm, vias 0 -> 3
- net Net-(J1-Pin_5): track 0.00 -> 36.6 mm
- net Net-(D8-A): track 0.00 -> 32.5 mm, vias 0 -> 2
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- added copper zone on B.Cu, net GND
Other:
- outline, holes or cut-outs redrawn
