File: control_unit/control_unit.kicad_pcb (KiCad board)
At the start: 2 copper layers, 100 x 95 mm, 114 parts, among them J2 Conn_01x02_Socket, J4 SERVO_PWM, J9 Barrel_Jack_Switch, Q3 2N7002, Q4 MMBT5551L, Q7 AO3400A, Q8 AO3400A, U1 CL6808, U14 MCP2515-xSO, U15 BNO055 DIP, U3 ATA6561-GAQW-N, U4 ADS1015IDGS, X1 16MHz

Commit message: 制御基板REV01完成
Parts:
- removed the D2 at (86.8, 129.6)
- removed the G*** at (167.5, 69.8)
- removed the Q4 at (164.7, 81.8)
- removed the R1 at (94.3, 128.8)
- removed the R16 at (130.5, 119.6)
- removed the R19 at (161.0, 80.6)
- removed SCL1, SDA1: SolderJumper_2_Open, Jumper:SolderJumper-2_P1.3mm_Open_RoundedPad1.0x1.5mm
- removed the TP1 at (124.3, 106.3)
- removed U15: BNO055 DIP, myfootprint:BNO055 DIP
- removed the U5 at (116.2, 112.0)
- added D1: SS36, Diode_SMD:D_SMA, F.Cu at (85.2, 129.8)
- added G***: LOGO, specific_footprint_library:aqua_logo, F.Cu at (166.4, 72.3)
- added JP1: SolderJumper_2_Bridged, Jumper:SolderJumper-2_P1.3mm_Bridged_RoundedPad1.0x1.5mm, F.Cu at (138.8, 101.2)
- added JP2: SolderJumper_2_Bridged, Jumper:SolderJumper-2_P1.3mm_Bridged_RoundedPad1.0x1.5mm, F.Cu at (138.8, 98.3)
- added Q3: 2N7002, Package_TO_SOT_SMD:SOT-23, F.Cu at (129.8, 118.0)
- added Q5: 2N7002, Package_TO_SOT_SMD:SOT-23, F.Cu at (165.0, 81.8)
- added R15: 100m, Resistor_SMD:R_1206_3216Metric, F.Cu at (159.2, 117.5)
- added R2: 100m, Resistor_SMD:R_1206_3216Metric, F.Cu at (91.0, 125.4)
- added R3: 100m, Resistor_SMD:R_1206_3216Metric, F.Cu at (91.0, 127.8)
- added R4: 100m, Resistor_SMD:R_1206_3216Metric, F.Cu at (91.0, 130.2)
- added R5: 100m, Resistor_SMD:R_1206_3216Metric, F.Cu at (91.0, 132.5)
- added R9: 1.2k, Resistor_SMD:R_0603_1608Metric_Pad0.98x0.95mm_HandSolder, F.Cu at (132.5, 119.5)
- added U1: ~, specific_footprint_library:VQFN-20_L4.5-W3.5-P0.50-BL-EP, F.Cu at (116.2, 112.0)
- added U7: BNO055 DIP, specific_footprint_library:BNO055 DIP, F.Cu at (148.2, 99.7)
- Cc1: renamed from Cc3; value 1500p -> 2.2n
- Cc2: value 82p -> 12p
- Cc3: renamed from Cc1; value 5.6n -> 3.3n
- L1: renamed from L3; footprint basic_parts:IND-SMD_L13.8-W12.6 -> specific_footprint_library:IND-SMD_L13.8-W12.6
- L2: footprint basic_parts:IND-SMD_L13.8-W12.6 -> specific_footprint_library:IND-SMD_L13.8-W12.6
- LED1: renamed from PWR1; value GREEN -> Emerald
- LED_PCB1: footprint Connector_JST:JST_XA_B06B-XASK-1_1x06_P2.50mm_Vertical -> Connector_JST:JST_XA_B06B-XASK-1-A_1x06_P2.50mm_Vertical
- R11: renamed from R12; value 5.1k -> 13k
- R12: renamed from R13; value 5.1k -> 3k
- R16: renamed from R17; value 1k -> 10k
- R18: renamed from R20; value 100k -> 10k
- Rc1: renamed from Rc2; value 560 -> 470
- Rc2: renamed from Rc1; value 10k -> 13k
- U3: renamed from U2; footprint basic_parts:Raspberry Pi 4 hat -> specific_footprint_library:RaspberryPi4 hat
- USER_LED1: value RED -> YELLOW
- X1: footprint basic_parts:OSC-SMD_4P-L3.2-W2.5-BL -> specific_footprint_library:OSC-SMD_4P-L3.2-W2.5-BL
- moved Rpg1 13.5 mm to (127.0, 119.5), turned to 180 degrees
- moved TP2 12.1 mm to (100.5, 116.2)
- moved Fan1 4.45 mm to (100.0, 109.7)
- moved U2 4.33 mm to (160.2, 112.2)
- moved D2 4.24 mm to (164.8, 112.2)
- moved R18 3.78 mm to (164.6, 79.2), turned to 180 degrees
- moved R14 3.18 mm to (161.6, 117.5), turned to -90 degrees
- moved J6 2.82 mm to (94.6, 96.6)
- moved LED_ESC_4 2.80 mm to (160.2, 133.5), turned to 0 degrees
- moved ESC4 2.28 mm to (160.5, 124.0)
- moved LED_ESC_3 2.15 mm to (156.5, 133.5), turned to 0 degrees
- moved LED_PCB1 1.78 mm to (166.5, 120.8)
- moved LED_BNO1 1.77 mm to (147.9, 106.5), turned to 0 degrees
- moved R1 1.70 mm to (149.2, 131.8), turned to 0 degrees
- moved LED_ESC_2 1.57 mm to (152.8, 133.5), turned to 0 degrees
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- renumbered C3 to C1, C5 to C3, C1 to C4, C4 to C5, D8 to D2, H5 to H2, H2 to H3, H6 to H4, H3 to H5, H4 to H6, J9 to J1, J4 to J3, Analog_IN1 to J4, CAN1 to J5, CAN2 to J6, JP1 to JP3, Q8 to Q1, Q7 to Q2, Q3 to Q4, Q1 to Q6, Q2 to Q7, R2 to R1, R4 to R10, R11 to R13, R10 to R14, R5 to R17, R14 to R19, R9 to R20, R8 to R21, R7 to R22, R6 to R23, R15 to R24, R21 to R6, R3 to R7, R18 to R8, TP2 to TP1, TP4 to TP2, U1 to U2, U14 to U4, U3 to U5, U4 to U6
Connections:
- net BLDC1_RP4 renamed ESC1_RP4
- net BLDC2_RP4 renamed ESC2_RP4
- net BLDC3_RP4 renamed ESC3_RP4
- net BLDC4_RP4 renamed ESC4_RP4
- LED1 pad 1: GND -> Net-(LED1-K)
- R14 pad 2: Net-(LED_PCB1-Pin_4) -> Net-(R14-Pad2)
- R18 pad 2: Net-(Q4-B) -> HighBeam
- Rpg1 pad 1: PGOOD -> Net-(Q3-G)
- Rpg1 pad 2: +3.3V_2 -> +5.1V
Routing:
- net PGOOD: track 24.1 -> 0.00 mm, vias 4 -> 0
- net Net-(Q3-G): track 0.00 -> 20.9 mm, vias 0 -> 5
- net +3.3V_2: track 85.1 -> 74.7 mm, vias 5 -> 3
- net Net-(D1-K): track 0.00 -> 9.54 mm
- net ESC1_RP4: track 72.9 -> 64.8 mm
- net Net-(Q4-B): track 5.80 -> 0.00 mm
- net ESC4_RP4: track 98.3 -> 93.4 mm
- net HighBeam: track 31.0 -> 35.8 mm
- net ESC3_RP4: track 87.1 -> 82.8 mm
- net ESC2_RP4: track 84.2 -> 80.4 mm
- net Net-(LED_PCB1-Pin_5): track 44.2 -> 47.4 mm
- net Net-(D2-K): track 2.97 -> 0.00 mm
- net +5.1V: track 205.6 -> 208.0 mm
- net Net-(R14-Pad2): track 0.00 -> 2.40 mm
- net Net-(Q4-D): track 40.0 -> 37.8 mm
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Other:
- board text added: "(GPIO26)"
- board text added: "(Lipo 3~12S)"
- board text added: "5.1V LB IR HB_A HB_K GND"
- board text added: "5.1V OK"
- board text added: "BNO 2.5V"
- board text added: "CANH"
- board text added: "CANL"
- board text added: "Don't input J1 & J2 simultaneously."
- board text added: "ESC1 GPIO21 ESC2 GPIO19 ESC3 GPIO16 ESC4 GPIO12"
- board text added: "ESC2"
- board text added: "ESC3"
- board text added: "ESC4"
- board text added: "FAN"
- board text added: "GND 5.1V PWM"
- board text added: "GND 5V PWM"
- board text added: "GPIO24"
- board text added: "HB GPIO5 LB GPIO6 IR GPIO25"
- board text added: "If not needed, please cut the heatsink area with a PCB cutter."
- board text added: "J2"
- board text added: "Please connect {dblquote}headlight_lower_side_pcb{dblquote} here before mounting the Raspberry Pi 4."
- board text added: "Please use either XA or XH for J3, J4, and J5."
- board text added: "RaspberryPi4 DCDC & CAN Hat"
- board text added: "SERVO DIRECT"
- board text added: "To headlight lower side"
- board text added: "Vin: 9V~45V"
- board text added: "When not using the ESC port, please jumper the PWM and 5V to use ESC1 to ESC4 as indicator LEDs."
- board text added: "↑High beam brightness"
- board text removed: "-"
- board text removed: "PWRGOOD"

Commit message: ESC周りの配線用基板進捗
Parts:
- removed R13: 10k, basic_parts:RES-ADJ-SMD_GF063P1
- added RV1: 10k, specific_footprint_library:TSR-3386, F.Cu at (157.2, 86.0)
- U5: footprint ATA6561:SOIC8_4P9X3P9MC_MCH -> specific_footprint_library:SOIC8_4P9X3P9MC_MCH
- moved R11 3.11 mm to (156.5, 92.8), turned to 90 degrees
- moved R18 2.87 mm to (161.8, 79.5), turned to -90 degrees
- moved C5 2.68 mm to (142.8, 93.2)
- moved JP3 1.39 mm to (147.5, 91.2)
- moved C1 1.36 mm to (151.0, 82.8)
- moved R_CAN1 1.35 mm to (148.8, 88.7)
- moved R12 1.32 mm to (159.2, 80.0), turned to 0 degrees
- moved C2 1.15 mm to (151.2, 76.8)
- moved X1 1.15 mm to (151.2, 79.8)
- moved U5 1.10 mm to (141.5, 89.7)
- moved U4 0.83 mm to (143.2, 80.2)
- moved Q4 0.70 mm to (165.0, 85.0)
- moved Q2 0.62 mm to (161.5, 76.0)
- moved Q5 0.60 mm to (165.2, 81.2)
- moved C3 0.60 mm to (137.0, 89.8)
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Connections:
- J3 pad 1: SERVO4 -> SERVO1
- J3 pad 2: SERVO3 -> SERVO2
- J3 pad 3: SERVO2 -> SERVO3
- J3 pad 4: SERVO1 -> SERVO4
- U3 pad 33: SERVO1 -> SERVO4
- U3 pad 7: SERVO4 -> SERVO1
Routing:
- net SERVO4: track 27.3 -> 67.7 mm
- net SERVO1: track 67.7 -> 27.3 mm
- net SERVO2: track 38.9 -> 35.4 mm
- net CANL: track 74.6 -> 72.2 mm
- net Net-(R11-Pad2): track 2.22 -> 4.46 mm
- net Net-(R12-Pad1): track 2.61 -> 4.71 mm
- net Net-(Q4-D): track 37.8 -> 35.9 mm
- net +3.3V_2: track 74.7 -> 76.6 mm, vias 3 -> 7
- net ESC1_RP4: track 64.8 -> 66.5 mm
- net CANH: track 75.6 -> 74.0 mm
- net Net-(U4-OSC1): track 9.23 -> 10.6 mm
- net LowBeam: track 27.7 -> 26.8 mm
- net SERVO3: track 33.6 -> 34.5 mm
- net Net-(U4-OSC2): track 9.31 -> 10.1 mm
- net Net-(U4-TXCAN): track 4.05 -> 3.29 mm
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Other:
- board text added: "(G26)"
- board text added: "ESC1 G21 ESC2 G19 ESC3 G16 ESC4 G12"
- board text added: "G24"
- board text added: "SERVO1 G4"
- board text added: "SERVO2 G18"
- board text added: "SERVO3 G17"
- board text added: "SERVO4 G13"
- board text removed: "(GPIO26)"
- board text removed: "ESC1 GPIO21 ESC2 GPIO19 ESC3 GPIO16 ESC4 GPIO12"
- board text removed: "GPIO24"
