File: power_circuit_vesc_express(bms)/power_circuit_vesc_express(bms).kicad_sch (KiCad schematic)
At the start: 1 part, among them U1 ESP32-C3-WROOM-02

Commit message: 制御基板REV01完成
Parts:
- added J1, J2, J3, J4: Conn_01x02_Socket, symbol Connector:Conn_01x02_Socket
Other:
- moved on the sheet: U1
