File: AQUA_VESC/can.kicad_sch (KiCad schematic)
At the start: 4 parts, among them U5 TJA1051T-3

Commit message: AQUA VESC仮完成
Parts:
- renumbered U5 to U4
Changed lines of the file:
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@@
 		(dnp no)
 		(fields_autoplaced yes)
-		(property "Reference" "#PWR042"
+		(property "Reference" "#PWR038"
 			(at 73.66 73.66 0)
 			(effects
@@
 			(project ""
 				(path "/8ee9fd02-9bd5-4905-927f-d8ca1179f479/eb11b7f4-5630-4685-a47e-4261806aa6f8"
-					(reference "#PWR042")
+					(reference "#PWR038")
 					(unit 1)
 				)
@@
 		(dnp no)
 		(fields_autoplaced yes)
-		(property "Reference" "#PWR041"
+		(property "Reference" "#PWR037"
 			(at 73.66 27.94 0)
 			(effects
@@
 			(project ""
 				(path "/8ee9fd02-9bd5-4905-927f-d8ca1179f479/eb11b7f4-5630-4685-a47e-4261806aa6f8"
-					(reference "#PWR041")
+					(reference "#PWR037")
 					(unit 1)
 				)
@@
 		(dnp no)
 		(fields_autoplaced yes)
-		(property "Reference" "#PWR040"
+		(property "Reference" "#PWR036"
 			(at 60.96 73.66 0)
 			(effects
@@
 			(project "AQUA_VESC"
 				(path "/8ee9fd02-9bd5-4905-927f-d8ca1179f479/eb11b7f4-5630-4685-a47e-4261806aa6f8"
-					(reference "#PWR040")
+					(reference "#PWR036")
 					(unit 1)
 				)
@@
 		(dnp no)
 		(fields_autoplaced yes)
-		(property "Reference" "U5"
+		(property "Reference" "U4"
 			(at 75.8033 41.91 0)
 			(effects
@@
 			(project ""
 				(path "/8ee9fd02-9bd5-4905-927f-d8ca1179f479/eb11b7f4-5630-4685-a47e-4261806aa6f8"
-					(reference "U5")
+					(reference "U4")
 					(unit 1)
 				)
@@
 		(dnp no)
 		(fields_autoplaced yes)
-		(property "Reference" "#PWR043"
+		(property "Reference" "#PWR039"
 			(at 80.01 41.91 0)
 			(effects
@@
 			(project "AQUA_VESC"
 				(path "/8ee9fd02-9bd5-4905-927f-d8ca1179f479/eb11b7f4-5630-4685-a47e-4261806aa6f8"
-					(reference "#PWR043")
+					(reference "#PWR039")
 					(unit 1)
 				)
@@
 		(dnp no)
 		(fields_autoplaced yes)
-		(property "Reference" "#PWR039"
+		(property "Reference" "#PWR035"
 			(at 48.26 59.69 0)
 			(effects
@@
 			(project ""
 				(path "/8ee9fd02-9bd5-4905-927f-d8ca1179f479/eb11b7f4-5630-4685-a47e-4261806aa6f8"
-					(reference "#PWR039")
-					(unit 1)
-				)
+					(reference "#PWR035")
+					(unit 1)
+				)

Commit message: 制御基板REV01完成
Parts:
- renumbered JP1 to JP2
Changed lines of the file:
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@@
 		(dnp no)
 		(fields_autoplaced yes)
-		(property "Reference" "#PWR038"
+		(property "Reference" "#PWR037"
 			(at 73.66 73.66 0)
 			(effects
@@
 			(project ""
 				(path "/8ee9fd02-9bd5-4905-927f-d8ca1179f479/eb11b7f4-5630-4685-a47e-4261806aa6f8"
-					(reference "#PWR038")
+					(reference "#PWR037")
 					(unit 1)
 				)
@@
 		(dnp no)
 		(fields_autoplaced yes)
-		(property "Reference" "#PWR037"
+		(property "Reference" "#PWR036"
 			(at 73.66 27.94 0)
 			(effects
@@
 			(project ""
 				(path "/8ee9fd02-9bd5-4905-927f-d8ca1179f479/eb11b7f4-5630-4685-a47e-4261806aa6f8"
-					(reference "#PWR037")
+					(reference "#PWR036")
 					(unit 1)
 				)
@@
 		(dnp no)
 		(fields_autoplaced yes)
-		(property "Reference" "JP1"
+		(property "Reference" "JP2"
 			(at 100.33 48.2599 90)
 			(effects
@@
 			(project ""
 				(path "/8ee9fd02-9bd5-4905-927f-d8ca1179f479/eb11b7f4-5630-4685-a47e-4261806aa6f8"
-					(reference "JP1")
+					(reference "JP2")
 					(unit 1)
 				)
@@
 		(dnp no)
 		(fields_autoplaced yes)
-		(property "Reference" "#PWR036"
+		(property "Reference" "#PWR035"
 			(at 60.96 73.66 0)
 			(effects
@@
 			(project "AQUA_VESC"
 				(path "/8ee9fd02-9bd5-4905-927f-d8ca1179f479/eb11b7f4-5630-4685-a47e-4261806aa6f8"
-					(reference "#PWR036")
+					(reference "#PWR035")
 					(unit 1)
 				)
@@
 		(dnp no)
 		(fields_autoplaced yes)
-		(property "Reference" "#PWR039"
+		(property "Reference" "#PWR038"
 			(at 80.01 41.91 0)
 			(effects
@@
 			(project "AQUA_VESC"
 				(path "/8ee9fd02-9bd5-4905-927f-d8ca1179f479/eb11b7f4-5630-4685-a47e-4261806aa6f8"
-					(reference "#PWR039")
+					(reference "#PWR038")
 					(unit 1)
 				)
@@
 		(dnp no)
 		(fields_autoplaced yes)
-		(property "Reference" "#PWR035"
+		(property "Reference" "#PWR034"
 			(at 48.26 59.69 0)
 			(effects
@@
 			(project ""
 				(path "/8ee9fd02-9bd5-4905-927f-d8ca1179f479/eb11b7f4-5630-4685-a47e-4261806aa6f8"
-					(reference "#PWR035")
-					(unit 1)
-				)
+					(reference "#PWR034")
+					(unit 1)
+				)
