File: AQUA_VESC-to-relay-pcb/AQUA_VESC-to-relay-pcb.kicad_pcb (KiCad board)
At the start: 2 copper layers, 102.1 x 80.5 mm, 11 parts, among them J1 Conn_01x04_Pin, J10 Conn_01x03_Pin, J2 Conn_01x04_Pin, J3 Conn_01x04_Pin, J4 Conn_01x04_Pin, J5 Conn_01x16_Pin, J6 Conn_01x12_Pin, J7 Conn_01x03_Pin, J8 Conn_01x03_Pin, J9 Conn_01x03_Pin

Commit message: ESC周りの配線用基板進捗
Parts:
- J5: footprint Connector_PinHeader_2.54mm:PinHeader_1x16_P2.54mm_Vertical -> Connector_PinSocket_2.54mm:PinSocket_1x16_P2.54mm_Vertical
- J6: footprint Connector_PinHeader_2.54mm:PinHeader_1x12_P2.54mm_Vertical -> Connector_PinSocket_2.54mm:PinSocket_1x12_P2.54mm_Vertical
- moved J10 0.60 mm to (90.9, 50.4)
- moved J4 0.60 mm to (90.9, 119.0)
- moved J9 0.40 mm to (114.9, 50.4)
- moved J3 0.40 mm to (114.9, 119.0)
- moved J8 0.20 mm to (138.9, 50.4)
- moved J2 0.20 mm to (138.9, 119.0)
Routing:
- net Net-(J6-Pin_10): track 110.9 -> 120.7 mm
- net Net-(J6-Pin_7): track 85.9 -> 82.3 mm
- net Net-(J6-Pin_11): track 111.1 -> 109.5 mm
- net Net-(J6-Pin_8): track 88.7 -> 87.3 mm
- net Net-(J4-Pin_1): track 24.6 -> 25.8 mm
- net Net-(J6-Pin_9): track 82.8 -> 81.8 mm
- net Net-(J6-Pin_4): track 52.0 -> 52.9 mm, vias 1 -> 0
- net Net-(J4-Pin_3): track 24.6 -> 25.2 mm
- net Net-(J10-Pin_2): track 24.6 -> 25.2 mm
- net Net-(J10-Pin_1): track 24.6 -> 25.2 mm
- net Net-(J6-Pin_12): track 112.8 -> 113.4 mm
- net Net-(J4-Pin_4): track 24.6 -> 25.2 mm
- net Net-(J4-Pin_2): track 24.6 -> 25.2 mm
Other:
- board size 102.1 x 80.5 mm -> 102 x 83.7 mm
