File: back_connector_base/back_connector_base.kicad_sch (KiCad schematic)
At the start: 10 parts, among them J1 Conn_01x12_Pin, J10 Conn_01x04_Socket, J2 Conn_01x16_Pin, J3 Conn_01x03_Socket, J4 Conn_01x03_Socket, J5 Conn_01x03_Socket, J6 Conn_01x03_Socket, J7 Conn_01x04_Socket, J8 Conn_01x04_Socket, J9 Conn_01x04_Socket

Commit message: ESC周りの配線用基板進捗
Parts:
- added H1, H2, H3: MountingHole, MountingHole:MountingHole_3.2mm_M3, symbol Mechanical:MountingHole
- added J11, J12: Conn_01x04_Pin, Connector_JST:JST_XH_B4B-XH-A_1x04_P2.50mm_Vertical, symbol Connector:Conn_01x04_Pin
- added J13: Conn_01x06_Pin, Connector_JST:JST_XH_B6B-XH-A_1x06_P2.50mm_Vertical, symbol Connector:Conn_01x06_Pin
- added JP1: SolderJumper_2_Bridged, Jumper:SolderJumper-2_P1.3mm_Bridged_RoundedPad1.0x1.5mm, symbol Jumper:SolderJumper_2_Bridged
- added R1: 120, Resistor_THT:R_Axial_DIN0207_L6.3mm_D2.5mm_P10.16mm_Horizontal, symbol Device:R
Connections:
- new net: J12.2 (Pin_2), J13.5 (Pin_5)
- new net: J12.3 (Pin_3), J13.6 (Pin_6)
- new net: J11.2 (Pin_2), J13.2 (Pin_2), R1.2
- new net: J11.3 (Pin_3), J13.3 (Pin_3), JP1.2 (B)
- new net: JP1.1 (A), R1.1
- new net +5V: J11.1 (Pin_1), J12.1 (Pin_1), J13.1 (Pin_1)
- new net GND: J11.4 (Pin_4), J12.4 (Pin_4), J13.4 (Pin_4)
Other:
- note added: "CAN"
- note added: "I2C"
- title: back_connector_cover -> back_connector_base
- moved on the sheet: J1, J10, J2, J3, J4, J5, J6, J7, J8, J9
