File: back_connector_esc/back_connector_esc.kicad_pcb (KiCad board)
At the start: 2 copper layers, 22 x 44 mm, 8 parts, among them J2 Conn_02x08_Odd_Even, J3 Conn_02x08_Odd_Even, J4 Conn_02x08_Odd_Even

Commit message: ESC周りの配線用基板進捗
Parts:
- removed G***: LOGO, specific_footprint_library:aqua_rogo
- removed MT60_Female: MT60F, specific_footprint_library:MT60_female
- moved H2 14.8 mm to (33.8, 55.2)
- moved H1 10.4 mm to (29.2, 50.2)
- moved H3 10.4 mm to (38.2, 50.2)
Other:
- board size 22 x 44 mm -> 22 x 33 mm
- board text removed: "REV00"
