File: can_connector/can_connector.kicad_pcb (KiCad board)
At the start: 2 copper layers, 102 x 35.6 mm, 16 parts, among them J1 Conn_01x02_Pin, J2 Conn_01x04_Pin, J3 Conn_01x02_Pin, J4 Conn_01x04_Pin, J5 Conn_01x02_Pin, J6 Conn_01x02_Pin, M1 Fan, M2 Fan

Commit message: ESC周りの配線用基板進捗
Parts:
- removed the J2 at (43.0, 49.0)
- added H5: MountingHole, MountingHole:MountingHole_3.2mm_M3, B.Cu at (83.0, 58.6)
- added H6: MountingHole, MountingHole:MountingHole_3.2mm_M3, B.Cu at (83.0, 78.6)
- added H7: MountingHole, MountingHole:MountingHole_3.2mm_M3, B.Cu at (103.0, 58.6)
- added H8: MountingHole, MountingHole:MountingHole_3.2mm_M3, B.Cu at (103.0, 78.6)
- added J6: Conn_01x06_Pin, Connector_PinHeader_2.54mm:PinHeader_1x06_P2.54mm_Vertical, F.Cu at (135.6, 49.0)
- added M3: Fan, Connector_PinHeader_2.54mm:PinHeader_1x02_P2.54mm_Vertical, B.Cu at (128.4, 49.0)
- J1: value Conn_01x02_Pin -> Conn_01x06_Pin; footprint Connector_PinHeader_2.54mm:PinHeader_1x02_P2.54mm_Vertical -> Connector_PinHeader_2.54mm:PinHeader_1x06_P2.54mm_Vertical; moved to B.Cu
- J4: value Conn_01x04_Pin -> Conn_01x02_Pin; footprint Connector_PinHeader_2.54mm:PinHeader_1x04_P2.54mm_Vertical -> Connector_PinHeader_2.54mm:PinHeader_1x02_P2.54mm_Vertical
- moved J2 92.0 mm to (43.6, 51.5)
- moved H12 33.7 mm to (130.0, 78.6)
- moved M1 29.5 mm to (75.1, 49.0), turned to -90 degrees
- moved H4 29.3 mm to (76.0, 78.6)
- moved H11 21.7 mm to (130.0, 58.6)
- moved H3 20.5 mm to (76.0, 58.6)
- moved H1 18.2 mm to (56.0, 58.6)
- moved H9 12.6 mm to (110.0, 58.6)
- moved M2 11.5 mm to (104.2, 49.0), turned to -90 degrees
- moved H10 7.41 mm to (110.0, 78.6)
- moved J1 2.63 mm to (38.6, 49.0), turned to 180 degrees
- moved J4 2.55 mm to (91.6, 51.5)
- moved H2 1.84 mm to (56.0, 78.6)
- moved J3 0.40 mm to (67.6, 51.5)
- renumbered H7 to H10, H4 to H11, H8 to H12, H5 to H2, H2 to H3, H6 to H4, H3 to H9, J6 to J2
Connections:
- J1 pad 1: CANH -> +5V
- J1 pad 2: CANL -> CANH
- J4 pad 1: Net-(J4-Pin_1) -> CANH
- J4 pad 2: CANH -> CANL
- M1 pad 1: Net-(J2-Pin_1) -> +5V
- M1 pad 2: Net-(J2-Pin_4) -> GND
- M2 pad 1: Net-(J4-Pin_1) -> +5V
- M2 pad 2: Net-(J4-Pin_4) -> GND
Routing:
- net SDA: track 0.00 -> 128.4 mm
- net SCL: track 0.00 -> 124.5 mm
- net GND: track 0.00 -> 112.3 mm
- net +5V: track 0.00 -> 104.9 mm
- net Net-(J2-Pin_1): track 10.7 -> 0.00 mm
- net Net-(J4-Pin_1): track 9.91 -> 0.00 mm
- net Net-(J2-Pin_4): track 6.28 -> 0.00 mm
- net Net-(J4-Pin_4): track 5.81 -> 0.00 mm
- net CANL: track 98.5 -> 102.5 mm
Other:
- outline, holes or cut-outs redrawn
- board text added: "CANH"
- board text added: "CANL"
- board text added: "SCL"
- board text added: "SDA"
