File: can_connector/can_connector.kicad_sch (KiCad schematic)
At the start: 16 parts, among them J1 Conn_01x02_Pin, J2 Conn_01x04_Pin, J3 Conn_01x02_Pin, J4 Conn_01x04_Pin, J5 Conn_01x02_Pin, J6 Conn_01x02_Pin, M1 Fan, M2 Fan

Commit message: ESC周りの配線用基板進捗
Parts:
- removed J1: Conn_01x02_Pin, Connector_PinHeader_2.54mm:PinHeader_1x02_P2.54mm_Vertical, symbol Connector:Conn_01x02_Pin
- removed J2, J4: Conn_01x04_Pin, Connector_PinHeader_2.54mm:PinHeader_1x04_P2.54mm_Vertical, symbol Connector:Conn_01x04_Pin
- added H5, H6, H7, H8: MountingHole, MountingHole:MountingHole_3.2mm_M3, symbol Mechanical:MountingHole
- added J1: Conn_01x06_Pin, Connector_PinHeader_2.54mm:PinHeader_1x06_P2.54mm_Vertical, symbol Connector:Conn_01x06_Pin
- added J4: Conn_01x02_Pin, Connector_PinHeader_2.54mm:PinHeader_1x02_P2.54mm_Vertical, symbol Connector:Conn_01x02_Pin
- added J6: Conn_01x06_Pin, Connector_JST_additonal:JST_XH_S6B-XH-A-1_1x06_P2.50mm_Horizontal, symbol Connector:Conn_01x06_Pin
- added M3: Fan, Connector_PinHeader_2.54mm:PinHeader_1x02_P2.54mm_Vertical, symbol Motor:Fan
- renumbered H7 to H10, H4 to H11, H8 to H12, H5 to H2, H2 to H3, H6 to H4, H3 to H9, J6 to J2
Connections:
- net CANH: now also J1.2 (Pin_2), J4.1 (Pin_1), J6.2 (Pin_2)
- net CANL: now also J1.3 (Pin_3), J4.2 (Pin_2), J6.3 (Pin_3)
- net +5V: now reaches M1.1 (+)
- net +5V: now also M2.1 (+), J1.1 (Pin_1), J6.1 (Pin_1), M3.1 (+)
- net GND: now reaches M1.2 (-)
- net GND: now also M2.2 (-), J1.4 (Pin_4), J6.4 (Pin_4), M3.2 (-)
- new net SCL: J1.6 (Pin_6), J6.6 (Pin_6)
- new net SDA: J1.5 (Pin_5), J6.5 (Pin_5)
Other:
- moved on the sheet: H1, H10, H11, H12, H2, H3, H4, H9, J2, M1, M2
